File: 7segLED6Digits/schematic.brd (EAGLE design)
At the start: 100 x 80 mm, 66 parts, among them Q1 MPSA56-TO92, Q2 MPSA56-TO92, Q3 MPSA56-TO92, Q4 MPSA56-TO92, Q5 MPSA56-TO92, Q6 MPSA56-TO92, T1 2SC1815, T10 2SC1815, T11 2SC1815, T12 2SC1815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

Commit message: ユニバーサル回路追加
Routing:
- net GND: track 0.00 -> 199.8 mm
- net N$7: track 0.00 -> 126.5 mm
- net SEGMENT6: track 0.00 -> 97.3 mm
- net SEGMENT7: track 0.00 -> 97.3 mm
- net SEGMENT1: track 0.00 -> 97.2 mm
- net SEGMENT2: track 0.00 -> 92.7 mm
- net SEGMENT5: track 0.00 -> 89.7 mm
- net SEGMENT3: track 0.00 -> 87.8 mm
- net SEGMENT4: track 0.00 -> 85.0 mm
- net N$8: track 0.00 -> 38.5 mm
- net N$39: track 0.00 -> 38.4 mm
- net N$45: track 0.00 -> 32.6 mm
- net N$19: track 0.00 -> 28.4 mm
- net N$11: track 0.00 -> 25.8 mm
- net N$40: track 0.00 -> 25.7 mm
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